Commit message: edit model

File: src/armoncar_package/urdf/mrobot_with_arm_and_laser.urdf.xacro (robot description, xacro)
@@ -1,4 +1,6 @@
 <?xml version="1.0"?>
-<robot name="mrobot" xmlns:xacro="http://www.ros.org/wiki/xacro">
+<robot xmlns:xacro="http://www.ros.org/wiki/xacro" name="panda_on_car">
+  <xacro:arg name="robot_name" default="panda"/>
+  <xacro:arg name="enable_rgdb_camera" default="true"/>
     <xacro:include filename="$(find armoncar_package)/urdf/mrobot_body.urdf.xacro" />
     <xacro:include filename="$(find armoncar_package)/urdf/rplidar.xacro" />
@@ -24,32 +26,4 @@
     <!-- Constants -->
     <xacro:property name="M_PI" value="3.14159"/>
-    <!-- link1 properties -->
-    <xacro:property name="link1_width" value="0.03" />
-    <xacro:property name="link1_len" value="0.10" />
-    <!-- link2 properties -->
-    <xacro:property name="link2_width" value="0.03" />
-    <xacro:property name="link2_len" value="0.14" />
-    <!-- link3 properties -->
-    <xacro:property name="link3_width" value="0.03" />
-    <xacro:property name="link3_len" value="0.22" />
-    <!-- link4 properties -->
-    <xacro:property name="link4_width" value="0.025" />
-    <xacro:property name="link4_len" value="0.06" />
-    <!-- link5 properties -->
-    <xacro:property name="link5_width" value="0.03" />
-    <xacro:property name="link5_len" value="0.06" />
-    <!-- link6 properties -->
-    <xacro:property name="link6_width" value="0.04" />
-    <xacro:property name="link6_len" value="0.02" />
-    <!-- Left gripper -->
-    <xacro:property name="left_gripper_len" value="0.08" />
-    <xacro:property name="left_gripper_width" value="0.01" />
-    <xacro:property name="left_gripper_height" value="0.01" />
-    <!-- Right gripper -->
-    <xacro:property name="right_gripper_len" value="0.08" />
-    <xacro:property name="right_gripper_width" value="0.01" />
-    <xacro:property name="right_gripper_height" value="0.01" />
-    <!-- Gripper frame -->
-    <xacro:property name="grasp_frame_radius" value="0.001" />
     <!-- Inertial matrix -->
     <xacro:macro name="inertial_matrix" params="mass">
@@ -59,5 +33,5 @@
         </inertial>
     </xacro:macro>
-    <!-- MRobot机器人平台-->
+    <!-- MRobot platform-->
     <mrobot_body/>
     <!-- rplidar -->
@@ -69,240 +43,21 @@
     <xacro:rplidar prefix="laser"/>
     <!-- arm -->
-    <joint name="arm_joint" type="fixed">
-        <origin xyz="${arm_offset_x} ${arm_offset_y} ${arm_offset_z}" rpy="0 0 0" />
-        <parent link="plate_2_link"/>
-        <child link="base_link_of_arm"/>
-    </joint>
-    <!-- ///////////////////////////////////////   bottom_joint   ////////////////////////////////////////// -->
-    <!--joint name="bottom_joint" type="fixed">
-        <origin xyz="0 0 0" rpy="0 0 0" />
-        <parent link="base_link_of_arm"/>
-        <child link="bottom_link"/>
-    </joint>
-    <link name="bottom_link">
-        <visual>
-              <origin xyz=" 0 0 -0.02"  rpy="0 0 0"/>
-                  <geometry>
-                       <box size="1 1 0.02" />
-                  </geometry>
-              <material name="Brown" />
-        </visual>
-        <collision>
-            <origin xyz=" 0 0 -0.02"  rpy="0 0 0"/>
-            <geometry>
-                <box size="1 1 0.02" />
-            </geometry>
-        </collision>
-        <xacro:inertial_matrix mass="500"/>
-    </link-->
-    <!-- /////////////////////////////////////   BASE LINK    ////////////////////////////////////////////// -->
-    <link name="base_link_of_arm">
-        <visual>
-            <origin xyz="0 0 0" rpy="0 0 0" />
-            <geometry>
-                <box size="0.1 0.1 0.04" />
-            </geometry>
-            <material name="White" />
-        </visual>
-        <collision>
-            <origin xyz="0 0 0" rpy="0 0 0" />
-            <geometry>
-                <box size="0.1 0.1 0.04" />
-            </geometry>
-        </collision>
-        <xacro:inertial_matrix mass="1"/>
-    </link>
-    <joint name="joint1" type="revolute">
-        <parent link="base_link_of_arm"/>
-        <child link="link1"/>
-        <origin xyz="0 0 0.02" rpy="0 ${M_PI/2} 0" />
-        <axis xyz="-1 0 0" />
-        <limit effort="300" velocity="1" lower="-2.96" upper="2.96"/>
-        <dynamics damping="50" friction="1"/>
-    </joint>
-    <!-- /////////////////////////////////////   LINK1  ////////////////////////////////////////////// -->
-    <link name="link1" >
-        <visual>
-            <origin xyz="-${link1_len/2} 0 0" rpy="0 ${M_PI/2} 0" />
-            <geometry>
-                <cylinder radius="${link1_width}" length="${link1_len}"/>
-            </geometry>
-            <material name="Blue" />
-        </visual>
-        <collision>
-            <origin xyz="-${link1_len/2} 0 0" rpy="0 ${M_PI/2} 0" />
-            <geometry>
-                <cylinder radius="${link1_width}" length="${link1_len}"/>
-            </geometry>
-        </collision>
-        <xacro:inertial_matrix mass="1"/>
-    </link>
-    <joint name="joint2" type="revolute">
-        <parent link="link1"/>
-        <child link="link2"/>
-        <origin xyz="-${link1_len} 0 0.0" rpy="-${M_PI/2} 0 ${M_PI/2}" />
-        <axis xyz="1 0 0" />
-        <limit effort="300" velocity="1.5" lower="-2.35" upper="2.35" />
-        <dynamics damping="50" friction="1"/>
-    </joint>
-    <!-- ///////////////////////////////////////   LINK2  ////////////////////////////////////////////// -->
-    <link name="link2" >
-        <visual>
-            <origin xyz="0 0 ${link2_len/2}" rpy="0 0 0" />
-            <geometry>
-                <cylinder radius="${link2_width}" length="${link2_len}"/>
-            </geometry>
-            <material name="White" />
-        </visual>
-        <collision>
-            <origin xyz="0 0 ${link2_len/2}" rpy="0 0 0" />
-            <geometry>
-                <cylinder radius="${link2_width}" length="${link2_len}"/>
-            </geometry>
-        </collision>
-        <xacro:inertial_matrix mass="1"/>
-    </link>
-    <joint name="joint3" type="revolute">
-        <parent link="link2"/>
-        <child link="link3"/>
-        <origin xyz="0 0 ${link2_len}" rpy="0 ${M_PI} 0" />
-        <axis xyz="-1 0 0" />
-        <limit effort="300" velocity="1" lower="-2.62" upper="2.62" />
-        <dynamics damping="50" friction="1"/>
-    </joint>
-    <!-- /////////////////////////////////   LINK3  ///////////////////////////////////////////////////// -->
-    <link name="link3" >
-        <visual>
-            <origin xyz="0 0 -${link3_len/2}" rpy="0 0 0" />
-            <geometry>
-                <cylinder radius="${link3_width}" length="${link3_len}"/>
-            </geometry>
-            <material name="Blue" />
-        </visual>
-        <collision>
-            <origin xyz="0 0 -${link3_len/2}" rpy="0 0 0" />
-            <geometry>
-                <cylinder radius="${link3_width}" length="${link3_len}"/>
-            </geometry>
-        </collision>
-        <xacro:inertial_matrix mass="1"/>
-    </link>
-    <joint name="joint4" type="revolute">
-        <parent link="link3"/>
-        <child link="link4"/>
-        <origin xyz="0.0 0.0 -${link3_len}" rpy="0 ${M_PI/2} ${M_PI}" />
-        <axis xyz="1 0 0" />
-        <limit effort="300" velocity="1" lower="-2.62" upper="2.62" />
-        <dynamics damping="50" friction="1"/>
-    </joint>
-    <!-- ///////////////////////////////////   LINK4  //////////////////////////////////////////////// -->
-    <link name="link4" >
-        <visual>
-            <origin xyz="${link4_len/2} 0 0" rpy="0 ${M_PI/2} 0" />
-            <geometry>
-                <cylinder radius="${link4_width}" length="${link4_len}"/>
-            </geometry>
-            <material name="Black" />
-        </visual>
-        <collision>
-            <origin xyz="${link4_len/2} 0 0" rpy="0 ${M_PI/2} 0" />
-            <geometry>
-                <cylinder radius="${link4_width}" length="${link4_len}"/>
-            </geometry>
-        </collision>
-        <xacro:inertial_matrix mass="1"/>
-    </link>
-    <joint name="joint5" type="revolute">
-        <parent link="link4"/>
-        <child link="link5"/>
-        <origin xyz="${link4_len} 0.0 0.0" rpy="0 ${M_PI/2} 0" />
-        <axis xyz="1 0 0" />
-        <limit effort="300" velocity="1" lower="-2.62" upper="2.62" />
-        <dynamics damping="50" friction="1"/>
-    </joint>
-    <!-- //////////////////////////////////   LINK5  ///////////////////////////////////////////////// -->
-    <link name="link5">
-        <visual>
-            <origin xyz="0 0 ${link4_len/2}" rpy="0 0 0" />
-            <geometry>
-                <cylinder radius="${link5_width}" length="${link5_len}"/>
-            </geometry>
-            <material name="White" />
-        </visual>
-        <collision>
-            <origin xyz="0 0 ${link4_len/2} " rpy="0 0 0" />
-            <geometry>
-                <cylinder radius="${link5_width}" length="${link5_len}"/>
-            </geometry>
-        </collision>
-        <xacro:inertial_matrix mass="1"/>
-    </link>
-    <joint name="joint6" type="revolute">
-        <parent link="link5"/>
-        <child link="link6"/>
-        <origin xyz="0 0 ${link4_len}" rpy="${1.5*M_PI} -${M_PI/2} 0" />
-        <axis xyz="1 0 0" />
-        <limit effort="300" velocity="1" lower="-6.28" upper="6.28" />
-        <dynamics damping="50" friction="1"/>
-    </joint>
-    <!-- ////////////////////////////////   LINK6  ///////////////////////////////////////////////// -->
-    <link name="link6">
-        <visual>
-            <origin xyz="${link6_len/2} 0 0 " rpy="0 ${M_PI/2} 0" />
-            <geometry>
-                <cylinder radius="${link6_width}" length="${link6_len}"/>
-            </geometry>
-            <material name="Blue" />
-        </visual>
-        <collision>
-            <origin xyz="${link6_len/2} 0 0" rpy="0 ${M_PI/2} 0" />
-            <geometry>
-                <cylinder radius="${link6_width}" length="${link6_len}"/>
-            </geometry>
-        </collision>
-        <xacro:inertial_matrix mass="1"/>
-    </link>
-    <joint name="finger_joint1" type="prismatic">
-        <parent link="link6"/>
-        <child link="gripper_finger_link1"/>
-        <origin xyz="0.0 0 0" />
-        <axis xyz="0 1 0" />
-        <limit effort="100" lower="0" upper="0.06" velocity="1.0"/>
-        <dynamics damping="50" friction="1"/>
-    </joint>
-    <!-- //////////////////////////////////////   gripper   ////////////////////////////////////////////// -->
-    <!-- LEFT GRIPPER AFT LINK -->
-    <link name="gripper_finger_link1">
-        <visual>
-            <origin xyz="0.04 -0.03 0"/>
-            <geometry>
-                <box size="${left_gripper_len} ${left_gripper_width} ${left_gripper_height}" />
-            </geometry>
-            <material name="White" />
-        </visual>
-        <xacro:inertial_matrix mass="1"/>
-    </link>
-    <joint name="finger_joint2" type="fixed">
-        <parent link="link6"/>
-        <child link="gripper_finger_link2"/>
-        <origin xyz="0.0 0 0" />
-    </joint>
-    <!-- RIGHT GRIPPER AFT LINK -->
-    <link name="gripper_finger_link2">
-        <visual>
-            <origin xyz="0.04 0.03 0"/>
-            <geometry>
-                <box size="${right_gripper_len} ${right_gripper_width} ${right_gripper_height}" />
-            </geometry>
-            <material name="White" />
-        </visual>
-        <xacro:inertial_matrix mass="1"/>
-    </link>
-    <!-- Grasping frame -->
-    <link name="grasping_frame"/>
-    <joint name="grasping_frame_joint" type="fixed">
-      <parent link="link6"/>
-      <child link="grasping_frame"/>
-      <origin xyz="0.08 0 0" rpy="0 0 0"/>
-    </joint>
+  <xacro:include filename="$(find easy_panda_sim)/robots/panda_arm.xacro"/>
+  <xacro:panda_arm />
+  <!-- gripper -->
+  <xacro:include filename="$(find easy_panda_sim)/robots/hand.xacro"/>
+  <xacro:hand rpy="0 0 ${-pi/4}" robot_name="$(arg robot_name)" connected_to="panda_link8"/>
+  <!-- additional gazebo tags -->
+  <xacro:include filename="$(find easy_panda_sim)/robots/panda.gazebo.xacro"/>
+  <xacro:panda_gazebo robot_name="$(arg robot_name)" />
+  <!-- gazebo HW interfaces -->
+  <xacro:include filename="$(find easy_panda_sim)/robots/panda.transmission.xacro"/>
+  <xacro:panda_transmission robot_name="$(arg robot_name)" />
+  <!-- RGB-D camera -->
+  <xacro:if value="$(arg enable_rgbd_camera)">
+    <xacro:include filename="$(find easy_panda_sim)/robots/rgbd_camera.xacro"/>
+    <xacro:rgbd_camera robot_name="$(arg robot_name)" />
+    <xacro:include filename="$(find easy_panda_sim)/robots/rgbd_camera.gazebo.xacro"/>
+    <xacro:rgbd_camera_gazebo robot_name="$(arg robot_name)" />
+  </xacro:if>
 </robot>
