Commit message: updates

File: src/armoncar_package/urdf/mrobot_body.urdf.xacro (robot description, xacro)
@@ -68,5 +68,5 @@
         <link name="base_link">
             <inertial>
-                <mass value="2" />
+                <mass value="200" />
                 <origin xyz="0 0 0.0" />
                 <inertia ixx="0.01" ixy="0.0" ixz="0.0"

File: src/armoncar_package/urdf/mrobot_with_arm_and_laser.urdf.xacro (robot description, xacro)
@@ -44,4 +44,6 @@
     <!-- arm -->
   <xacro:include filename="$(find easy_panda_sim)/robots/panda_arm.xacro"/>
+  <xacro:include filename="$(find armoncar_package)/urdf/panda.control.xacro"/>
+  <xacro:panda_control arm_id="panda"/>
   <xacro:panda_arm />
   <!-- gripper -->

Commit message: new updates

File: src/armoncar_package/urdf/mrobot_body.urdf.xacro (robot description, xacro)
@@ -1,17 +1,144 @@
 <?xml version="1.0"?>
-<robot xmlns:xacro="http://www.ros.org/wiki/xacro">
-    <xacro:property name="M_PI" value="3.14159"/>
-    <xacro:property name="wheel_radius" value="0.033"/>
-    <xacro:property name="wheel_length" value="0.017"/>
+<robot name="mrobot" xmlns:xacro="http://www.ros.org/wiki/xacro">
+    <!-- PROPERTY LIST -->
+    <!-- Main body length, width, height and mass -->
+    <xacro:property name="base_mass"        value="200" />
     <xacro:property name="base_link_radius" value="0.13"/>
     <xacro:property name="base_link_length" value="0.005"/>
-    <xacro:property name="motor_radius" value="0.02"/>
-    <xacro:property name="motor_length" value="0.08"/>
-    <xacro:property name="motor_x" value="-0.055"/>
-    <xacro:property name="motor_y" value="0.075"/>
+    <xacro:property name="motor_x" value="-0.05"/>
+    <!-- Caster radius and mass -->
+    <xacro:property name="caster_radius"          value="0.016" />
+    <xacro:property name="caster_mass"            value="0.01" />
+    <xacro:property name="caster_joint_origin_x"  value="-0.12" />
+    <!-- Wheel radius, height and mass -->
+    <xacro:property name="wheel_radius" value="0.033" />
+    <xacro:property name="wheel_height" value="0.017" />
+    <xacro:property name="wheel_mass"   value="0.1" />
+    <!-- plate height and mass -->
+    <xacro:property name="plate_mass"   value="0.05"/>
     <xacro:property name="plate_height" value="0.07"/>
-    <xacro:property name="standoff_x" value="0.12"/>
-    <xacro:property name="standoff_y" value="0.10"/>
-    <!-- 定义MRobot本体的宏 -->
+    <xacro:property name="standoff_x"   value="0.12"/>
+    <xacro:property name="standoff_y"   value="0.10"/>
+    <!-- Macro for inertia matrix -->
+    <xacro:macro name="sphere_inertial_matrix" params="m r">
+        <inertial>
+            <mass value="${m}" />
+            <inertia ixx="${2*m*r*r/5}" ixy="0" ixz="0"
+                iyy="${2*m*r*r/5}" iyz="0"
+                izz="${2*m*r*r/5}" />
+        </inertial>
+    </xacro:macro>
+    <xacro:macro name="cylinder_inertial_matrix" params="m r h">
+        <inertial>
+            <mass value="${m}" />
+            <inertia ixx="${m*(3*r*r+h*h)/12}" ixy = "0" ixz = "0"
+                iyy="${m*(3*r*r+h*h)/12}" iyz = "0"
+                izz="${m*r*r/2}" />
+        </inertial>
+    </xacro:macro>
+    <xacro:macro name="box_inertial_matrix" params="m w h d">
+        <inertial>
+            <mass value="${m}" />
+            <inertia ixx="${m*(h*h+d*d)/12}" ixy = "0" ixz = "0"
+                iyy="${m*(w*w+d*d)/12}" iyz = "0"
+                izz="${m*(w*w+h*h)/12}" />
+        </inertial>
+    </xacro:macro>
+    <!-- Macro for wheel joint -->
+    <xacro:macro name="wheel" params="lr translateY">
+        <!-- lr: left, right -->
+        <link name="wheel_${lr}_link">
+            <visual>
+                <origin xyz="0 0 0" rpy="${M_PI/2} 0  0 " />
+                <geometry>
+                    <cylinder length="${wheel_height}" radius="${wheel_radius}" />
+                </geometry>
+                <material name="Black" />
+            </visual>
+            <collision>
+                <origin xyz="0 0 0" rpy="${M_PI/2} 0 0 " />
+                <geometry>
+                    <cylinder length="${wheel_height}" radius="${wheel_radius}" />
+                </geometry>
+            </collision>
+            <cylinder_inertial_matrix  m="${wheel_mass}" r="${wheel_radius}" h="${wheel_height}" />
+        </link>
+        <gazebo reference="wheel_${lr}_link">
+            <material>Gazebo/Black</material>
+        </gazebo>
+        <joint name="base_to_wheel_${lr}_joint" type="continuous">
+            <parent link="base_link"/>
+            <child link="wheel_${lr}_link"/>
+            <origin xyz="${motor_x} ${translateY * base_link_radius} 0" rpy="0 0 0" />
+            <axis xyz="0 1 0" rpy="0  0" />
+        </joint>
+        <!-- Transmission is important to link the joints and the controller -->
+        <transmission name="wheel_${lr}_joint_trans">
+            <type>transmission_interface/SimpleTransmission</type>
+            <joint name="base_to_wheel_${lr}_joint">
+		<hardwareInterface>hardware_interface/EffortJointInterface</hardwareInterface>
+	    </joint>
+            <actuator name="wheel_${lr}_joint_motor">
+                <hardwareInterface>VelocityJointInterface</hardwareInterface>
+                <mechanicalReduction>1</mechanicalReduction>
+            </actuator>
+        </transmission>
+    </xacro:macro>
+    <!-- Macro for caster joint -->
+    <xacro:macro name="caster" params="fb translateX">
+        <!-- fb: front, back -->
+        <link name="${fb}_caster_link">
+            <visual>
+                <origin xyz="0 0 0 " rpy="0 0 0" />
+                <geometry>
+                    <sphere radius="${caster_radius}" />
+                </geometry>
+                <material name="Black" />
+            </visual>
+            <collision>
+                <geometry>
+                    <sphere radius="${caster_radius}" />
+                </geometry>
+                <origin xyz="0 0 0 " rpy="0 0 0" />
+            </collision>
+            <sphere_inertial_matrix  m="${caster_mass}" r="${caster_radius}" />
+        </link>
+        <gazebo reference="${fb}_caster_link">
+            <material>Gazebo/Black</material>
+        </gazebo>
+        <joint name="base_to_${fb}_caster_joint" type="fixed">
+            <parent link="base_link"/>
+            <child link="${fb}_caster_link"/>
+            <origin xyz="${translateX*caster_joint_origin_x} 0 ${-caster_radius}" rpy="0 0 0"/>
+        </joint>
+    </xacro:macro>
+    <!-- Macro for plate joint -->
+    <xacro:macro name="plate" params="num parent">
+        <link name="plate_${num}_link">
+            <cylinder_inertial_matrix  m="0.1" r="${base_link_radius}" h="${base_link_length}" />
+            <visual>
+                <origin xyz=" 0 0 0 " rpy="0 0 0" />
+                <geometry>
+                    <cylinder length="${base_link_length}" radius="${base_link_radius}"/>
+                </geometry>
+                <material name="yellow"/>
+            </visual>
+            <collision>
+                <origin xyz="0.0 0.0 0.0" rpy="0 0 0" />
+                <geometry>
+                    <cylinder length="${base_link_length}" radius="${base_link_radius}"/>
+                </geometry>
+            </collision>
+        </link>
+        <gazebo reference="plate_${num}_link">
+            <material>Gazebo/Blue</material>
+        </gazebo>
+        <joint name="plate_${num}_joint" type="fixed">
+            <origin xyz="0 0 ${plate_height}" rpy="0 0 0" />
+            <parent link="${parent}"/>
+            <child link="plate_${num}_link" />
+        </joint>
+    </xacro:macro>
+    <!-- Macro for standoff joint -->
     <xacro:macro name="mrobot_standoff_2in" params="parent number x_loc y_loc z_loc">
         <joint name="standoff_2in_${number}_joint" type="fixed">
@@ -25,6 +152,6 @@
                 <origin xyz="0 0 0" />
                 <inertia ixx="0.0001" ixy="0.0" ixz="0.0"
-                         iyy="0.0001" iyz="0.0"
-                         izz="0.0001" />
+          iyy="0.0001" iyz="0.0"
+          izz="0.0001" />
             </inertial>
             <visual>
@@ -45,17 +172,7 @@
         </link>
     </xacro:macro>
+    <!-- BASE-FOOTPRINT -->
+    <!-- base_footprint is a fictitious link(frame) that is on the ground right below base_link origin -->
     <xacro:macro name="mrobot_body">
-        <material name="Green">
-            <color rgba="0.0 0.8 0.0 1.0"/>
-        </material>
-        <material name="yellow">
-            <color rgba="1 0.4 0 1"/>
-        </material>
-        <material name="black">
-            <color rgba="0 0 0 0.95"/>
-        </material>
-        <material name="gray">
-            <color rgba="0.75 0.75 0.75 1"/>
-        </material>
         <link name="base_footprint">
             <visual>
@@ -65,25 +182,4 @@
                 </geometry>
             </visual>
-        </link>
-        <link name="base_link">
-            <inertial>
-                <mass value="200" />
-                <origin xyz="0 0 0.0" />
-                <inertia ixx="0.01" ixy="0.0" ixz="0.0"
-                         iyy="0.01" iyz="0.0" izz="0.5" />
-            </inertial>
-            <visual>
-                <origin xyz=" 0 0 0" rpy="0 0 0" />
-                <geometry>
-                    <cylinder length="${base_link_length}" radius="${base_link_radius}"/>
-                </geometry>
-                <material name="yellow" />
-            </visual>
-            <collision>
-                <origin xyz="0 0 0" rpy="0 0 0" />
-                <geometry>
-                    <cylinder length="${base_link_length}" radius="${base_link_radius}"/>
-                </geometry>
-            </collision>
         </link>
         <joint name="base_footprint_joint" type="fixed">
@@ -92,200 +188,66 @@
             <child link="base_link" />
         </joint>
-        <link name="left_motor">
-            <inertial>
-                <origin xyz="0.0 0 0"/>
-                <mass value="0.1" />
-                <inertia ixx="0.001" ixy="0.0" ixz="0.0"
-                         iyy="0.001" iyz="0.0" izz="0.001" />
-            </inertial>
-            <visual>
-                <origin xyz="0 0 0" rpy="${M_PI/2} 0 0" />
-                <geometry>
-                    <cylinder radius="${motor_radius}" length = "${motor_length}"/>
-                </geometry>
-                <material name="gray" />
-            </visual>
-            <collision>
-                <origin xyz="0 0 0" rpy="${M_PI/2} 0 0" />
-                <geometry>
-                    <cylinder radius="${motor_radius}" length = "${motor_length}"/>
-                </geometry>
-            </collision>
-        </link>
-        <joint name="base_left_motor_joint" type="fixed">
-            <origin xyz="${motor_x} ${motor_y} 0" rpy="0 0 0" />
-            <parent link="base_link"/>
-            <child link="left_motor" />
-        </joint>
-        <link name="left_wheel_link">
-            <inertial>
-                <origin xyz="0 0 0"/>
-                <mass value="0.01" />
-                <inertia ixx="0.001" ixy="0.0" ixz="0.0"
-                         iyy="0.001" iyz="0.0" izz="0.001" />
-            </inertial>
-            <visual>
-                <origin xyz="0 0 0" rpy="${M_PI/2} 0 0" />
-                <geometry>
-                    <cylinder radius="${wheel_radius}" length = "${wheel_length}"/>
-                </geometry>
-                <material name="white">
-                    <color rgba="1 1 1 0.9"/>
-                </material>
-            </visual>
-            <collision>
-                <origin xyz="0 0 0" rpy="${M_PI/2} 0 0" />
-                <geometry>
-                    <cylinder radius="${wheel_radius}" length = "${wheel_length}"/>
-                </geometry>
-            </collision>
-        </link>
-        <joint name="left_wheel_joint" type="continuous">
-            <origin xyz="0 ${(motor_length+wheel_length)/2} 0" rpy="0 0 0"/>
-            <parent link="left_motor"/>
-            <child link="left_wheel_link"/>
-            <axis xyz="0 1 0"/>
-        </joint>
-        <link name="right_motor">
-            <inertial>
-                <origin xyz="0.0 0 0"/>
-                <mass value="0.1" />
-                <inertia ixx="0.001" ixy="0.0" ixz="0.0"
-                         iyy="0.001" iyz="0.0" izz="0.001" />
-            </inertial>
-            <visual>
-                <origin xyz="0 0 0" rpy="${M_PI/2} 0 0" />
-                <geometry>
-                    <cylinder radius="${motor_radius}" length = "${motor_length}" />
-                </geometry>
-                <material name="gray" />
-            </visual>
-            <collision>
-                <origin xyz="0 0 0" rpy="${M_PI/2} 0 0" />
-                <geometry>
-                    <cylinder radius="${motor_radius}" length = "${motor_length}"/>
-                </geometry>
-            </collision>
-        </link>
-        <joint name="base_right_motor_joint" type="fixed">
-            <origin xyz="${motor_x} -${motor_y} 0" rpy="0 0 0" />
-            <parent link="base_link"/>
-            <child link="right_motor" />
-        </joint>
-        <link name="right_wheel_link">
-            <inertial>
-                <origin xyz="0 0 0"/>
-                <mass value="0.01" />
-                <inertia ixx="0.001" ixy="0.0" ixz="0.0"
-                         iyy="0.001" iyz="0.0" izz="0.001" />
-            </inertial>
-            <visual>
-                <origin xyz="0 0 0" rpy="${M_PI/2} 0 0" />
-                <geometry>
-                    <cylinder radius="${wheel_radius}" length = "${wheel_length}"/>
-                </geometry>
-                <material name="white">
-                    <color rgba="1 1 1 0.9"/>
-                </material>
-            </visual>
-            <collision>
-                <origin xyz="0 0 0" rpy="${M_PI/2} 0 0" />
-                <geometry>
-                    <cylinder radius="${wheel_radius}" length = "${wheel_length}"/>
-                </geometry>
-            </collision>
-        </link>
-        <joint name="right_wheel_joint" type="continuous">
-            <origin xyz="0 -${(motor_length+wheel_length)/2} 0" rpy="0 0 0"/>
-            <parent link="right_motor"/>
-            <child link="right_wheel_link"/>
-            <axis xyz="0 1 0"/>
-        </joint>
-        <link name="front_caster_link">
-            <inertial>
-                <origin xyz="0 0 0"/>
-                <mass value="0.001" />
-                <inertia ixx="0.0001" ixy="0.0" ixz="0.0"
-                         iyy="0.0001" iyz="0.0" izz="0.0001" />
-            </inertial>
-            <visual>
-                <origin xyz="0 0 0" rpy="${M_PI/2} 0 0"/>
-                <geometry>
-                    <sphere radius="${wheel_radius/2}" />
-                </geometry>
-                <material name="black" />
-            </visual>
-            <collision>
-                <origin xyz="0 0 0.01" rpy="${M_PI/2} 0 0" />
-                <geometry>
-                    <sphere radius="${wheel_radius/2}" />
-                </geometry>
-            </collision>
-        </link>
-        <joint name="front_caster_joint" type="fixed">
-            <origin xyz="${base_link_radius-wheel_radius/2} 0 -${wheel_radius/2}" rpy="0 0 0"/>
-            <parent link="base_link"/>
-            <child link="front_caster_link"/>
-        </joint>
+        <!-- BASE-LINK -->
+        <!--Actual body/chassis of the robot-->
+        <link name="base_link">
+            <cylinder_inertial_matrix  m="${base_mass}" r="${base_link_radius}" h="${base_link_length}" />
+            <visual>
+                <origin xyz=" 0 0 0" rpy="0 0 0" />
+                <geometry>
+                    <cylinder length="${base_link_length}" radius="${base_link_radius}"/>
+                </geometry>
+                <material name="yellow" />
+            </visual>
+            <collision>
+                <origin xyz="0 0 0" rpy="0 0 0" />
+                <geometry>
+                    <cylinder length="${base_link_length}" radius="${base_link_radius}"/>
+                </geometry>
+            </collision>
+        </link>
+        <gazebo reference="base_link">
+            <material>Gazebo/Blue</material>
+        </gazebo>
+        <!-- Wheel Definitions -->
+        <wheel lr="right"  translateY="1" />
+        <wheel lr="left"  translateY="-1" />
+        <!-- Casters Definitions -->
+        <caster fb="front"  translateX="-1" />
+        <!-- plates and standoff Definitions -->
         <mrobot_standoff_2in parent="base_link" number="1" x_loc="-${standoff_x/2 + 0.03}" y_loc="-${standoff_y - 0.03}" z_loc="${plate_height/2}"/>
         <mrobot_standoff_2in parent="base_link" number="2" x_loc="-${standoff_x/2 + 0.03}" y_loc="${standoff_y - 0.03}" z_loc="${plate_height/2}"/>
         <mrobot_standoff_2in parent="base_link" number="3" x_loc="${standoff_x/2}" y_loc="-${standoff_y}" z_loc="${plate_height/2}"/>
         <mrobot_standoff_2in parent="base_link" number="4" x_loc="${standoff_x/2}" y_loc="${standoff_y}" z_loc="${plate_height/2}"/>
-        <joint name="plate_1_joint" type="fixed">
-            <origin xyz="0 0 ${plate_height}" rpy="0 0 0" />
-            <parent link="base_link"/>
-            <child link="plate_1_link" />
-        </joint>
-        <link name="plate_1_link">
-            <inertial>
-                <mass value="0.1" />
-                <origin xyz="0 0 0" />
-                <inertia ixx="0.01" ixy="0.0" ixz="0.0"
-                         iyy="0.01" iyz="0.0" izz="0.01" />
-            </inertial>
-            <visual>
-                <origin xyz=" 0 0 0 " rpy="0 0 0" />
-                <geometry>
-                    <cylinder length="${base_link_length}" radius="${base_link_radius}"/>
-                </geometry>
-                <material name="yellow"/>
-            </visual>
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
File: src/armoncar_package/urdf/mrobot_with_arm_and_laser.urdf.xacro (robot description, xacro)
@@ -43,22 +43,11 @@
     <xacro:rplidar prefix="laser"/>
     <!-- arm -->
-  <xacro:include filename="$(find easy_panda_sim)/robots/panda_arm.xacro"/>
-  <xacro:include filename="$(find armoncar_package)/urdf/panda.control.xacro"/>
-  <xacro:panda_control arm_id="panda"/>
-  <xacro:panda_arm />
-  <!-- gripper -->
-  <xacro:include filename="$(find easy_panda_sim)/robots/hand.xacro"/>
-  <xacro:hand rpy="0 0 ${-pi/4}" robot_name="$(arg robot_name)" connected_to="panda_link8"/>
-  <!-- additional gazebo tags -->
-  <xacro:include filename="$(find easy_panda_sim)/robots/panda.gazebo.xacro"/>
-  <xacro:panda_gazebo robot_name="$(arg robot_name)" />
-  <!-- gazebo HW interfaces -->
-  <xacro:include filename="$(find easy_panda_sim)/robots/panda.transmission.xacro"/>
-  <xacro:panda_transmission robot_name="$(arg robot_name)" />
+  <xacro:include filename="$(find armoncar_package)/urdf/robots/panda/panda.urdf.xacro"/>
+  <franka_panda/>
   <!-- RGB-D camera -->
   <xacro:if value="$(arg enable_rgbd_camera)">
-    <xacro:include filename="$(find easy_panda_sim)/robots/rgbd_camera.xacro"/>
+    <xacro:include filename="$(find armoncar_package)/urdf/robots/rgbd_camera/rgbd_camera.xacro"/>
     <xacro:rgbd_camera robot_name="$(arg robot_name)" />
-    <xacro:include filename="$(find easy_panda_sim)/robots/rgbd_camera.gazebo.xacro"/>
+    <xacro:include filename="$(find armoncar_package)/urdf/robots/rgbd_camera/rgbd_camera.gazebo.xacro"/>
     <xacro:rgbd_camera_gazebo robot_name="$(arg robot_name)" />
   </xacro:if>
