Commit message: new updates

File: src/armoncar_package/urdf/xxx.urdf (robot description, URDF)
Before this commit: robot panda_on_car, 34 links, 33 joints
Links:
- removed link left_motor
- removed link left_wheel_link
- removed link panda_tcp
- removed link right_motor
- removed link right_wheel_link
- added link panda_hand_sc; collision cylinder length=0.1 radius=0.05; collision cylinder length=0.1 radius=0.07
- added link panda_hand_tcp
- added link panda_link0_sc; collision cylinder length=0.03 radius=0.09; collision sphere radius=0.09
- added link panda_link1_sc; collision cylinder length=0.283 radius=0.09; collision sphere radius=0.09
- added link panda_link2_sc; collision cylinder length=0.12 radius=0.09; collision sphere radius=0.09
- added link panda_link3_sc; collision cylinder length=0.15 radius=0.09; collision sphere radius=0.09
- added link panda_link4_sc; collision cylinder length=0.12 radius=0.09; collision sphere radius=0.09
- added link panda_link5_sc; collision cylinder length=0.1 radius=0.09; collision cylinder length=0.14 radius=0.055
- added link panda_link6_sc; collision cylinder length=0.08 radius=0.08; collision sphere radius=0.08
- added link panda_link7_sc; collision cylinder length=0.01 radius=0.06; collision cylinder length=0.14 radius=0.07
- added link wheel_left_link, mass 0.1; collision cylinder length=0.017 radius=0.033; visual cylinder length=0.017 radius=0.033
- added link wheel_right_link, mass 0.1; collision cylinder length=0.017 radius=0.033; visual cylinder length=0.017 radius=0.033
- link front_caster_link: mass 0.001 -> 0.01; geometry collision sphere radius=0.016; visual sphere radius=0.016
- link panda_hand: mass 0.68 -> None; geometry collision mesh filename=package://franka_description/meshes/collision/hand.stl; visual mesh filename=package://franka_description/meshes/visual/hand.dae
- link panda_leftfinger: mass 0.01 -> None; geometry collision box size=17.5e-3 15.2e-3 18.5e-3; collision box size=17.5e-3 7e-3 23.5e-3
- link panda_link0: mass 3.06357 -> None; geometry collision mesh filename=package://franka_description/meshes/collision/link0.stl; visual mesh filename=package://franka_description/meshes/visual/link0.dae
- link panda_link1: mass 2.34471 -> None; geometry collision mesh filename=package://franka_description/meshes/collision/link1.stl; visual mesh filename=package://franka_description/meshes/visual/link1.dae
- link panda_link2: mass 2.36414 -> None; geometry collision mesh filename=package://franka_description/meshes/collision/link2.stl; visual mesh filename=package://franka_description/meshes/visual/link2.dae
- link panda_link3: mass 2.3805 -> None; geometry collision mesh filename=package://franka_description/meshes/collision/link3.stl; visual mesh filename=package://franka_description/meshes/visual/link3.dae
- link panda_link4: mass 2.42754 -> None; geometry collision mesh filename=package://franka_description/meshes/collision/link4.stl; visual mesh filename=package://franka_description/meshes/visual/link4.dae
- link panda_link5: mass 3.49611 -> None; geometry collision mesh filename=package://franka_description/meshes/collision/link5.stl; visual mesh filename=package://franka_description/meshes/visual/link5.dae
- link panda_link6: mass 1.46736 -> None; geometry collision mesh filename=package://franka_description/meshes/collision/link6.stl; visual mesh filename=package://franka_description/meshes/visual/link6.dae
- link panda_link7: mass 0.45606 -> None; geometry collision mesh filename=package://franka_description/meshes/collision/link7.stl; visual mesh filename=package://franka_description/meshes/visual/link7.dae
- link panda_link8: mass 0.001 -> None
- link panda_rgbd: geometry visual mesh filename=package://armoncar_package/urdf/meshes/visual/rgbd_camera.d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
- link panda_rightfinger: mass 0.01 -> None; geometry collision box size=17.5e-3 15.2e-3 18.5e-3; collision box size=17.5e-3 7e-3 23.5e-3
- link plate_2_link: mass 0.01 -> 0.1
Joints:
- removed joint base_left_motor_joint
- removed joint base_right_motor_joint
- removed joint front_caster_joint
- removed joint left_wheel_joint
- removed joint panda_tcp_joint
- removed joint right_wheel_joint
- removed joint robot_to_world
- added joint base_to_front_caster_joint: type fixed, parent base_link, child front_caster_link, origin xyz=0.12 0 -0.016 rpy=0 0 0
- added joint base_to_wheel_left_joint: type continuous, parent base_link, child wheel_left_link, origin xyz=-0.05 -0.13 0 rpy=0 0 0, axis 0 1 0
- added joint base_to_wheel_right_joint: type continuous, parent base_link, child wheel_right_link, origin xyz=-0.05 0.13 0 rpy=0 0 0, axis 0 1 0
- added joint panda_hand_sc_joint: type fixed, parent panda_hand, child panda_hand_sc, origin rpy=0 0 0
- added joint panda_hand_tcp_joint: type fixed, parent panda_hand, child panda_hand_tcp, origin xyz=0 0 0.1034 rpy=0 0 0
- added joint panda_joint_plate_2_link: type fixed, parent plate_2_link, child panda_link0, origin xyz=0 0 0 rpy=0 0 0
- added joint panda_link0_sc_joint: type fixed, parent panda_link0, child panda_link0_sc, origin rpy=0 0 0
- added joint panda_link1_sc_joint: type fixed, parent panda_link1, child panda_link1_sc, origin rpy=0 0 0
- added joint panda_link2_sc_joint: type fixed, parent panda_link2, child panda_link2_sc, origin rpy=0 0 0
- added joint panda_link3_sc_joint: type fixed, parent panda_link3, child panda_link3_sc, origin rpy=0 0 0
- added joint panda_link4_sc_joint: type fixed, parent panda_link4, child panda_link4_sc, origin rpy=0 0 0
- added joint panda_link5_sc_joint: type fixed, parent panda_link5, child panda_link5_sc, origin rpy=0 0 0
- added joint panda_link6_sc_joint: type fixed, parent panda_link6, child panda_link6_sc, origin rpy=0 0 0
- added joint panda_link7_sc_joint: type fixed, parent panda_link7, child panda_link7_sc, origin rpy=0 0 0.785398163397
- joint panda_finger_joint1: limit lower=0.0 upper=0.04 effort=20 velocity=0.2 -> lower=0.0 upper=0.04 effort=100 velocity=0.2
- joint panda_finger_joint2: limit lower=0.0 upper=0.04 effort=20 velocity=0.2 -> lower=0.0 upper=0.04 effort=100 velocity=0.2
- joint panda_joint1: limit lower=-2.8973 upper=2.8973 effort=87 velocity=2.1750 -> lower=-2.8973 upper=2.8973 effort=87.0 velocity=2.175
- joint panda_joint2: limit lower=-1.7628 upper=1.7628 effort=87 velocity=2.1750 -> lower=-1.7628 upper=1.7628 effort=87.0 velocity=2.175
- joint panda_joint3: limit lower=-2.8973 upper=2.8973 effort=87 velocity=2.1750 -> lower=-2.8973 upper=2.8973 effort=87.0 velocity=2.175
- joint panda_joint4: limit lower=-3.0718 upper=-0.0698 effort=87 velocity=2.1750 -> lower=-3.0718 upper=-0.0698 effort=87.0 velocity=2.175
- joint panda_joint5: limit lower=-2.8973 upper=2.8973 effort=12 velocity=2.6100 -> lower=-2.8973 upper=2.8973 effort=12.0 velocity=2.61
- joint panda_joint6: limit lower=-0.0175 upper=3.7525 effort=12 velocity=2.6100 -> lower=-0.0175 upper=3.7525 effort=12.0 velocity=2.61
- joint panda_joint7: limit lower=-2.8973 upper=2.8973 effort=12 velocity=2.6100 -> lower=-2.8973 upper=2.8973 effort=12.0 velocity=2.61
- joint panda_joint8: axis 0 0 1 -> (none); limit lower=0 upper=0.1 effort=1 velocity=0.1 -> (none)
